File: example_project/ESP32_C6_Dev_Board/ESP32_C6_Dev_Board.kicad_pcb (KiCad board)
At the start: 2 copper layers, 95 x 80 mm, 14 parts

Commit message: update readme
Parts:
- D1, D2, D3, J1, J2, U1, U2: value ~ -> (none)
- moved U1 132.8 mm to (9.40, 40.0)
- moved C1 128.9 mm to (6.00, 25.0)
- moved C2 128.9 mm to (20.5, 40.0)
- moved D1 128.4 mm to (6.00, 10.0)
- moved D2 127.7 mm to (6.00, 15.0)
- moved R2 127.1 mm to (6.00, 5.00)
- moved J1 120.4 mm to (10.0, 59.0)
- moved C3 120.4 mm to (28.9, 40.0)
- moved U2 92.6 mm to (40.0, 40.0)
- moved D3 87.6 mm to (52.2, 40.0)
- moved R3 79.6 mm to (60.5, 40.0)
- moved J2 73.9 mm to (40.6, 40.0)
- moved R1 49.0 mm to (76.7, 40.0)
- moved C4 43.2 mm to (68.7, 40.0)
Connections:
- C1 pad 1: /ESP32_C6_Dev_Board_Main/VBUS_OUT -> unconnected-(C1-Pad1-Pad1)
- C1 pad 2: /ESP32_C6_Dev_Board_Main/GND -> unconnected-(C1-Pad2-Pad2)
- C2 pad 1: /ESP32_C6_Dev_Board_Main/VBUS_IN -> unconnected-(C2-Pad1-Pad1)
- C2 pad 2: /ESP32_C6_Dev_Board_Main/GND -> unconnected-(C2-Pad2-Pad2)
- C3 pad 1: /ESP32_C6_Dev_Board_Main/VCC_3V3_OUT -> unconnected-(C3-Pad1-Pad1)
- C3 pad 2: /ESP32_C6_Dev_Board_Main/GND -> unconnected-(C3-Pad2-Pad2)
- C4 pad 1: /ESP32_C6_Dev_Board_Main/VCC_3V3 -> unconnected-(C4-Pad1-Pad1)
- C4 pad 2: /ESP32_C6_Dev_Board_Main/GND -> unconnected-(C4-Pad2-Pad2)
- D1 pad 1: /ESP32_C6_Dev_Board_Main/USB_DP -> unconnected-(D1-Pad1-Pad1)
- D1 pad 2: /ESP32_C6_Dev_Board_Main/GND -> unconnected-(D1-Pad2-Pad2)
- D2 pad 1: /ESP32_C6_Dev_Board_Main/USB_DM -> unconnected-(D2-Pad1-Pad1)
- D2 pad 2: /ESP32_C6_Dev_Board_Main/GND -> unconnected-(D2-Pad2-Pad2)
- D3 pad 1: /ESP32_C6_Dev_Board_Main/LED_CONTROL -> unconnected-(D3-Pad1-Pad1)
- D3 pad 2: /ESP32_C6_Dev_Board_Main/N$3 -> unconnected-(D3-Pad2-Pad2)
- J1 pad : (no net) -> unconnected-(J1-Pad-Pad)
- J1 pad A1: /ESP32_C6_Dev_Board_Main/GND -> unconnected-(J1-PadA1-PadA1)
- J1 pad A12: /ESP32_C6_Dev_Board_Main/GND -> unconnected-(J1-PadA12-PadA12)
- J1 pad A4: /ESP32_C6_Dev_Board_Main/VBUS_OUT -> unconnected-(J1-PadA4-PadA4)
- J1 pad A5: /ESP32_C6_Dev_Board_Main/N$1 -> unconnected-(J1-PadA5-PadA5)
- J1 pad A6: /ESP32_C6_Dev_Board_Main/USB_DP -> unconnected-(J1-PadA6-PadA6)
- J1 pad A7: /ESP32_C6_Dev_Board_Main/USB_DM -> unconnected-(J1-PadA7-PadA7)
- J1 pad A9: /ESP32_C6_Dev_Board_Main/VBUS_OUT -> unconnected-(J1-PadA9-PadA9)
- J1 pad B1: /ESP32_C6_Dev_Board_Main/GND -> unconnected-(J1-PadB1-PadB1)
- J1 pad B12: /ESP32_C6_Dev_Board_Main/GND -> unconnected-(J1-PadB12-PadB12)
- J1 pad B4: /ESP32_C6_Dev_Board_Main/VBUS_OUT -> unconnected-(J1-PadB4-PadB4)
- J1 pad B5: /ESP32_C6_Dev_Board_Main/N$2 -> unconnected-(J1-PadB5-PadB5)
- J1 pad B9: /ESP32_C6_Dev_Board_Main/VBUS_OUT -> unconnected-(J1-PadB9-PadB9)
- J1 pad S1: /ESP32_C6_Dev_Board_Main/GND -> unconnected-(J1-PadS1-PadS1)
- J2 pad 1: /ESP32_C6_Dev_Board_Main/DEBUG_EN -> unconnected-(J2-Pad1-Pad1)
- J2 pad 2: /ESP32_C6_Dev_Board_Main/VCC_3V3 -> unconnected-(J2-Pad2-Pad2)
- J2 pad 3: /ESP32_C6_Dev_Board_Main/DEBUG_TX -> unconnected-(J2-Pad3-Pad3)
- J2 pad 4: /ESP32_C6_Dev_Board_Main/GND -> unconnected-(J2-Pad4-Pad4)
- J2 pad 5: /ESP32_C6_Dev_Board_Main/DEBUG_RX -> unconnected-(J2-Pad5-Pad5)
- J2 pad 6: /ESP32_C6_Dev_Board_Main/DEBUG_IO0 -> unconnected-(J2-Pad6-Pad6)
- R1 pad 1: /ESP32_C6_Dev_Board_Main/N$1 -> unconnected-(R1-Pad1-Pad1)
- R1 pad 2: /ESP32_C6_Dev_Board_Main/GND -> unconnected-(R1-Pad2-Pad2)
- R2 pad 1: /ESP32_C6_Dev_Board_Main/N$2 -> unconnected-(R2-Pad1-Pad1)
- R2 pad 2: /ESP32_C6_Dev_Board_Main/GND -> unconnected-(R2-Pad2-Pad2)
- R3 pad 1: /ESP32_C6_Dev_Board_Main/VCC_3V3 -> unconnected-(R3-Pad1-Pad1)
- R3 pad 2: /ESP32_C6_Dev_Board_Main/N$3 -> unconnected-(R3-Pad2-Pad2)
- U1 pad 1: /ESP32_C6_Dev_Board_Main/GND -> unconnected-(U1-Pad1-Pad1)
- U1 pad 2: /ESP32_C6_Dev_Board_Main/VCC_3V3_OUT -> unconnected-(U1-Pad2-Pad2)
- U1 pad 3: /ESP32_C6_Dev_Board_Main/VBUS_IN -> unconnected-(U1-Pad3-Pad3)
- U2 pad 1: /ESP32_C6_Dev_Board_Main/GND -> unconnected-(U2-Pad1-Pad1)
- U2 pad 11: /ESP32_C6_Dev_Board_Main/GND -> unconnected-(U2-Pad11-Pad11)
- U2 pad 12: /ESP32_C6_Dev_Board_Main/DEBUG_IO0 -> unconnected-(U2-Pad12-Pad12)
- U2 pad 14: /ESP32_C6_Dev_Board_Main/GND -> unconnected-(U2-Pad14-Pad14)
- U2 pad 2: /ESP32_C6_Dev_Board_Main/GND -> unconnected-(U2-Pad2-Pad2)
- U2 pad 22: /ESP32_C6_Dev_Board_Main/LED_CONTROL -> unconnected-(U2-Pad22-Pad22)
- U2 pad 24: /ESP32_C6_Dev_Board_Main/USB_DP -> unconnected-(U2-Pad24-Pad24)
- U2 pad 25: /ESP32_C6_Dev_Board_Main/USB_DM -> unconnected-(U2-Pad25-Pad25)
- U2 pad 3: /ESP32_C6_Dev_Board_Main/VCC_3V3 -> unconnected-(U2-Pad3-Pad3)
- U2 pad 30: /ESP32_C6_Dev_Board_Main/DEBUG_RX -> unconnected-(U2-Pad30-Pad30)
- U2 pad 31: /ESP32_C6_Dev_Board_Main/DEBUG_TX -> unconnected-(U2-Pad31-Pad31)
- U2 pad 36: /ESP32_C6_Dev_Board_Main/GND -> unconnected-(U2-Pad36-Pad36)
- U2 pad 37: /ESP32_C6_Dev_Board_Main/GND -> unconnected-(U2-Pad37-Pad37)
- U2 pad 38: /ESP32_C6_Dev_Board_Main/GND -> unconnected-(U2-Pad38-Pad38)
- U2 pad 39: /ESP32_C6_Dev_Board_Main/GND -> unconnected-(U2-Pad39-Pad39)
- U2 pad 40: /ESP32_C6_Dev_Board_Main/GND -> unconnected-(U2-Pad40-Pad40)
- U2 pad 41: /ESP32_C6_Dev_Board_Main/GND -> unconnected-(U2-Pad41-Pad41)
- U2 pad 42: /ESP32_C6_Dev_Board_Main/GND -> unconnected-(U2-Pad42-Pad42)
- U2 pad 43: /ESP32_C6_Dev_Board_Main/GND -> unconnected-(U2-Pad43-Pad43)
- U2 pad 44: /ESP32_C6_Dev_Board_Main/GND -> unconnected-(U2-Pad44-Pad44)
- U2 pad 45: /ESP32_C6_Dev_Board_Main/GND -> unconnected-(U2-Pad45-Pad45)
- U2 pad 46: /ESP32_C6_Dev_Board_Main/GND -> unconnected-(U2-Pad46-Pad46)
- U2 pad 47: /ESP32_C6_Dev_Board_Main/GND -> unconnected-(U2-Pad47-Pad47)
- U2 pad 48: /ESP32_C6_Dev_Board_Main/GND -> unconnected-(U2-Pad48-Pad48)
- U2 pad 49: /ESP32_C6_Dev_Board_Main/GND -> unconnected-(U2-Pad49-Pad49)
- U2 pad 50: /ESP32_C6_Dev_Board_Main/GND -> unconnected-(U2-Pad50-Pad50)
- U2 pad 51: /ESP32_C6_Dev_Board_Main/GND -> unconnected-(U2-Pad51-Pad51)
- U2 pad 52: /ESP32_C6_Dev_Board_Main/GND -> unconnected-(U2-Pad52-Pad52)
- U2 pad 53: /ESP32_C6_Dev_Board_Main/GND -> unconnected-(U2-Pad53-Pad53)
- U2 pad 8: /ESP32_C6_Dev_Board_Main/DEBUG_EN -> unconnected-(U2-Pad8-Pad8)
