File: kicad_reference/kicad_reference.kicad_sch (KiCad schematic)
At the start: 1 part

Commit message: add docs and example
Parts:
- removed R1: 10k, Resistor_SMD:R_0603_1608Metric, symbol Device:R
- added U1: AMS1117-3.3, Package_TO_SOT_SMD:SOT-223-3_TabPin2, symbol Regulator_Linear:AMS1117-3.3
Changed lines of the file:
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@@
 	(paper "A4")
 	(symbol
-		(lib_id "Device:R")
-		(at 121.92 73.66 0)
+		(lib_id "Regulator_Linear:AMS1117-3.3")
+		(at 135.89 96.52 0)
 		(unit 1)
 		(exclude_from_sim no)
@@
 		(dnp no)
 		(fields_autoplaced yes)
-		(property "Reference" "R1"
-			(at 124.46 72.3899 0)
+		(property "Reference" "U1"
+			(at 135.89 90.17 0)
 			(effects
 				(font
 					(size 1.27 1.27)
 				)
-				(justify left)
 			)
 		)
-		(property "Value" "10k"
-			(at 124.46 74.9299 0)
+		(property "Value" "AMS1117-3.3"
+			(at 135.89 92.71 0)
 			(effects
 				(font
 					(size 1.27 1.27)
 				)
-				(justify left)
 			)
 		)
-		(property "Footprint" "Resistor_SMD:R_0603_1608Metric"
-			(at 120.142 73.66 90)
+		(property "Footprint" "Package_TO_SOT_SMD:SOT-223-3_TabPin2"
+			(at 135.89 91.44 0)
 			(effects
 				(font
@@
 			)
 		)
-		(property "Datasheet" "~"
-			(at 121.92 73.66 0)
+		(property "Datasheet" "http://www.advanced-monolithic.com/pdf/ds1117.pdf"
+			(at 138.43 102.87 0)
 			(effects
 				(font
@@
 			)
 		)
-		(property "Description" "Resistor"
-			(at 121.92 73.66 0)
+		(property "Description" "1A Low Dropout regulator, positive, 3.3V fixed output, SOT-223"
+			(at 135.89 96.52 0)
 			(effects
 				(font
@@
 		(pin "2"
 		)
+		(pin "3"
+		)
 		(instances
 			(project "kicad_reference"
-				(path "/7dc21ed6-d010-4774-8661-489ad2d53c39"
-					(reference "R1")
+				(path "/5f0ac341-7bbd-4a3f-be5f-8ffd62126d0c"
+					(reference "U1")
 					(unit 1)
 				)
