File: demos/02_esp32_devboard/ESP32_C6_Dev_Board/ESP32_C6_MCU.kicad_sch (KiCad schematic)
At the start: 4 parts

Commit message: remove uneeded files
Parts:
- added D3: (no value), LED_SMD:LED_0805_2012Metric, symbol Device:LED
- added J2: (no value), Connector_IDC:IDC-Header_2x03_P2.54mm_Vertical, symbol Connector_Generic:Conn_02x03_Odd_Even
- added R3: 330, Resistor_SMD:R_0805_2012Metric, symbol Device:R
Connections:
- net DEBUG_EN: now also J2.1 (Pin_1)
- net DEBUG_IO0: now also J2.6 (Pin_6)
- net DEBUG_RX: now also J2.5 (Pin_5)
- net DEBUG_TX: now also J2.3 (Pin_3)
- net GND: now also D3.1 (K), J2.4 (Pin_4)
- net LED_CONTROL: now also R3.1
- net N$3: now also D3.2 (A), R3.2
- net VCC_3V3: now also J2.2 (Pin_2)
