File: demos/02_esp32_devboard/ESP32_C6_Dev_Board/USB_Port.kicad_sch (KiCad schematic)
At the start: 6 parts

Commit message: remove uneeded files
Changed lines of the file:
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@@
 		)
 		(instances
-			(project "ESP32_C6_Dev_Board"
+			(project "b7723a2a-a62f-4d4b-ba05-2cd14f395e7c"
 				(path "/b7723a2a-a62f-4d4b-ba05-2cd14f395e7c/965f9aa0-87a0-4779-a8ee-b6c4c54bbb07"
 					(reference "J1")
@@
 		)
 		(instances
-			(project "ESP32_C6_Dev_Board"
+			(project "b7723a2a-a62f-4d4b-ba05-2cd14f395e7c"
 				(path "/b7723a2a-a62f-4d4b-ba05-2cd14f395e7c/965f9aa0-87a0-4779-a8ee-b6c4c54bbb07"
 					(reference "R1")
@@
 		)
 		(instances
-			(project "ESP32_C6_Dev_Board"
+			(project "b7723a2a-a62f-4d4b-ba05-2cd14f395e7c"
 				(path "/b7723a2a-a62f-4d4b-ba05-2cd14f395e7c/965f9aa0-87a0-4779-a8ee-b6c4c54bbb07"
 					(reference "R2")
@@
 		)
 		(instances
-			(project "ESP32_C6_Dev_Board"
+			(project "b7723a2a-a62f-4d4b-ba05-2cd14f395e7c"
 				(path "/b7723a2a-a62f-4d4b-ba05-2cd14f395e7c/965f9aa0-87a0-4779-a8ee-b6c4c54bbb07"
 					(reference "D1")
@@
 		)
 		(instances
-			(project "ESP32_C6_Dev_Board"
+			(project "b7723a2a-a62f-4d4b-ba05-2cd14f395e7c"
 				(path "/b7723a2a-a62f-4d4b-ba05-2cd14f395e7c/965f9aa0-87a0-4779-a8ee-b6c4c54bbb07"
 					(reference "D2")
@@
 		)
 		(instances
-			(project "ESP32_C6_Dev_Board"
+			(project "b7723a2a-a62f-4d4b-ba05-2cd14f395e7c"
 				(path "/b7723a2a-a62f-4d4b-ba05-2cd14f395e7c/965f9aa0-87a0-4779-a8ee-b6c4c54bbb07"
 					(reference "C1")
@@
 		)
 	)
-	(text_box
-		"USB-C port with CC resistors, ESD protection, and proper grounding"
-		(exclude_from_sim yes)
-		(at 184.0 110.0 0)
-		(size 80.0 30.0)
-		(margins
-			1.0
-			1.0
-			1.0
-			1.0
-		)
-		(stroke
-			(width 0.1)
-			(type solid)
-		)
-		(fill
-			(type color)
-			(color
-				255
-				255
-				224
-				1
-			)
-		)
-		(effects
-			(font
-				(size 1.2 1.2)
-				(thickness 0.254)
-			)
-			(justify left top)
-		)
-	)
 	(sheet_instances
-		(path "/b7723a2a-a62f-4d4b-ba05-2cd14f395e7c/965f9aa0-87a0-4779-a8ee-b6c4c54bbb07"
+		(path "/"
 			(page "1")
 		)
