File: reference_circuit-synth/reference_generated/reference_generated.kicad_sch (KiCad schematic)
At the start: 1 part

Commit message: Fix symbol 'at' expression format - always include angle for KiCad compatibility
- Modified s_expression.py to always include angle (even if 0) in symbol at expressions
- Changed from (at x y) to (at x y angle) format as required by KiCad
- Fixes 'need a number for symbol orientation' error when opening schematics
- Simplified formatter by removing old complex formatting logic with 15+ boolean flags
- Now using only clean, rule-based formatter (~1800 lines removed)
Connections:
- removed net GND: R1.2
Other:
- removed sheet child1
- company: Circuit-Synth -> (none)
- title: main -> (none)
Changed lines of the file:
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@@
 	(version 20250114)
 	(generator "circuit_synth")
-	(generator_version "9.0")
-	(paper "A4")
-	(title_block
-		(title main)
-		(date 2025-08-08)
-		(company Circuit-Synth)
-	)
 	(symbol
 		(lib_id "Device:R")
-		(at 38.1 45.72 0)
+		(at 38.1 40.64 0.0)
 		(unit 1)
 		(exclude_from_sim no)
@@
 		(dnp no)
 		(fields_autoplaced yes)
-		(property "Reference" "R1"
-			(at 38.1 40.72 0)
+		(property
+			"Reference"
+			"R1"
+			(at 38.1 35.64 0)
 			(effects
 				(font
@@
 			)
 		)
-		(property "Value" "R"
-			(at 38.1 50.72 0)
+		(property
+			"Value"
+			"R"
+			(at 38.1 45.64 0)
 			(effects
 				(font
@@
 		)
 		(instances
-			(project ""
-				(path "/e54f82e6-12e8-4c3f-acea-b4b89cde6221"
+			(project
+				"reference_generated"
+				(path
+					"/"
 					(reference "R1")
 					(unit 1)
@@
 		)
 	)
-	(hierarchical_label
-		GND
-		(shape input)
-		(at 38.1 49.53 270)
-		(effects
-			(font
-				(size 1.27 1.27)
-			)
-			(justify right)
-		)
-	)
-	(hierarchical_label
-		GND
-		(shape input)
-		(at 97.63 39.37 0)
-		(effects
-			(font
-				(size 1.27 1.27)
-			)
-			(justify left)
-		)
-	)
-	(sheet
-		(at 58.42 36.83)
-		(size 39.21 20.32)
-		(stroke
-			(width 0.12)
-			(type solid)
-		)
-		(fill
-			(color
-				0
-				0
-				0
-				0.0
-			)
-		)
-		(property "Sheetname" "child1"
-			(at 58.42 35.559999999999995 0)
-			(effects
-				(font
-					(size 1.27 1.27)
-				)
-				(justify left bottom)
-			)
-		)
-		(property "Sheetfile" "child1.kicad_sch"
-			(at 58.42 58.42 0)
-			(effects
-				(font
-					(size 1.27 1.27)
-				)
-				(justify left top)
-				(hide yes)
-			)
-		)
-		(pin
-			GND
-			passive
-			(at 96.36 39.37 0)
-			(effects
-				(font
-					(size 1.27 1.27)
-				)
-				(justify right)
-			)
-		)
-		(instances
-			(project "reference_generated"
-				(path "/"
-					(page "1")
-				)
-			)
-		)
-	)
-	(text_box
-		"Main circuit with hierarchical subcircuits"
-		(exclude_from_sim yes)
-		(at 184.0 110.0 0)
-		(size 80.0 30.0)
-		(margins
-			1.0
-			1.0
-			1.0
-			1.0
-		)
-		(stroke
-			(width 0.1)
-			(type solid)
-		)
-		(fill
-			(type color)
-			(color
-				255
-				255
-				224
-				1
-			)
-		)
-		(effects
-			(font
-				(size 1.2 1.2)
-				(thickness 0.254)
-			)
-			(justify left top)
-		)
-	)
-	(sheet_instances
-		(path "/e54f82e6-12e8-4c3f-acea-b4b89cde6221"
-			(page "1")
-		)
-	)
-	(embedded_fonts no)
 )

Commit message: Fix lib_symbols population with actual symbol definitions
- Added detailed logging to track lib_symbols generation
- lib_symbols now properly populated with symbol definitions from cache
- Symbol definitions include properties, graphics, and pin information
- Symbols now render correctly in KiCad instead of showing as ?? boxes
- Reference circuit now generates with complete symbol library data
Connections:
- new net GND: R1.2
Other:
- added sheet child1 (child1.kicad_sch)
Changed lines of the file:
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@@
 	(symbol
 		(lib_id "Device:R")
-		(at 38.1 40.64 0.0)
+		(at 38.1 45.72 0.0)
 		(unit 1)
 		(exclude_from_sim no)
@@
 			"Reference"
 			"R1"
-			(at 38.1 35.64 0)
+			(at 38.1 40.72 0)
 			(effects
 				(font
@@
 			"Value"
 			"R"
-			(at 38.1 45.64 0)
+			(at 38.1 50.72 0)
 			(effects
 				(font
@@
 		(instances
 			(project
-				"reference_generated"
+				""
 				(path
-					"/"
+					"/a2642601-3cef-41e9-a654-ec36e9238345"
 					(reference "R1")
 					(unit 1)
 				)
 			)
+		)
+	)
+	(hierarchical_label
+		"GND"
+		(shape
+			input
+		)
+		(at 38.1 49.53 270)
+		(effects
+			(font
+				(size 1.27 1.27)
+			)
+			(justify right)
+		)
+	)
+	(hierarchical_label
+		"GND"
+		(shape
+			input
+		)
+		(at 97.63 39.37 0)
+		(effects
+			(font
+				(size 1.27 1.27)
+			)
+			(justify left)
+		)
+	)
+	(sheet
+		(at 58.42 36.83)
+		(size 39.21 20.32)
+		(stroke
+			(width 0.12)
+			(type solid)
+		)
+		(fill
+			(color 0 0 0 0.0)
+		)
+		(property
+			"Sheetname"
+			"child1"
+			(at 58.42 35.559999999999995 0)
+			(effects
+				(font
+					(size 1.27 1.27)
+				)
+				(justify left bottom)
+			)
+		)
+		(property
+			"Sheetfile"
+			"child1.kicad_sch"
+			(at 58.42 58.42 0)
+			(effects
+				(font
+					(size 1.27 1.27)
+				)
+				(justify left top)
+				(hide yes)
+			)
+		)
+		(pin
+			GND
+			passive
+			(at 96.36 39.37 0)
+			(effects
+				(font
+					(size 1.27 1.27)
+				)
+				(justify right)
+			)
+		)
+		(instances
+			(project
+				"reference_generated"
+				(path
+					"/"
+					(page "1")
+				)
+			)
