File: tests/bidirectional/03_python_to_kicad/single_resistor/single_resistor.kicad_sch (KiCad schematic)
At the start: 1 part

Commit message: update tests
Parts:
- removed R1: 10k, Resistor_SMD:R_0603_1608Metric, symbol Device:R
Changed lines of the file:
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@@
 (kicad_sch
 	(version 20250114)
-	(generator "circuit_synth")
-	(generator_version "0.8.36")
+	(generator "eeschema")
+	(generator_version "9.0")
 	(paper "A4")
-	(symbol
-		(lib_id "Device:R")
-		(at 30.48 35.56 0)
-		(unit 1)
-		(exclude_from_sim no)
-		(in_bom yes)
-		(on_board yes)
-		(dnp no)
-		(fields_autoplaced yes)
-		(property "Reference" "R1"
-			(at 33.02 34.2899 0)
-			(effects
-				(font
-					(size 1.27 1.27)
-				)
-				(justify left)
-			)
-		)
-		(property "Value" "10k"
-			(at 33.02 36.8299 0)
-			(effects
-				(font
-					(size 1.27 1.27)
-				)
-				(justify left)
-			)
-		)
-		(property "Footprint" "Resistor_SMD:R_0603_1608Metric"
-			(at 28.702 35.56 90)
-			(effects
-				(font
-					(size 1.27 1.27)
-				)
-				(hide yes)
-			)
-		)
-		(property "hierarchy_path" "/9980990e-9d60-4586-8e99-cd1ffc9652d5"
-			(at 33.02 40.6399 0)
-			(effects
-				(font
-					(size 1.27 1.27)
-				)
-				(hide yes)
-			)
-		)
-		(property "project_name" "single_resistor"
-			(at 33.02 40.6399 0)
-			(effects
-				(font
-					(size 1.27 1.27)
-				)
-				(hide yes)
-			)
-		)
-		(property "root_uuid" "9980990e-9d60-4586-8e99-cd1ffc9652d5"
-			(at 33.02 40.6399 0)
-			(effects
-				(font
-					(size 1.27 1.27)
-				)
-				(hide yes)
-			)
-		)
-		(pin "1"
-		)
-		(pin "2"
-		)
-		(instances
-			(project "single_resistor"
-				(path "/9980990e-9d60-4586-8e99-cd1ffc9652d5"
-					(reference "R1")
-					(unit 1)
-				)
-			)
-		)
-	)
-	(text_box "Circuit with a single 10kΩ resistor."
-		(exclude_from_sim no)
-		(at 184 110 0)
-		(size 80 30)
-		(margins 1 1 1 1)
-		(stroke
-			(width 0)
-			(type solid)
-		)
-		(fill
-			(type none)
-		)
-		(effects
-			(font
-				(size 1.2 1.2)
-			)
-			(justify left top)
-		)
-	)
 	(sheet_instances
 		(path "/"
