File: tests/bidirectional/10_generate_with_net/two_resistors_connected/two_resistors_connected.kicad_sch (KiCad schematic)
At the start: 2 parts

Commit message: docs: Correct test 10 - hierarchical labels don't use wires
Fixed test 10 documentation to reflect correct KiCad behavior:
- Hierarchical labels with matching names establish electrical connection
- NO physical wires drawn between components
- Labels appear as square flags on component pins

Changes:
- Removed all references to 'wire connecting R1 to R2'
- Added 'NO physical wire' clarifications throughout
- Explained how matching label names create electrical connection
- Updated expected results to check for labels, not wires
- Simplified generate_kicad_project() call (no extra params)

This is correct KiCad behavior for hierarchical labels.
Parts:
- R1, R2: hierarchy_path /c2956866-50a0-4e52-8385-61296f5ada12 -> /27c31603-b2e8-4b1a-86a9-80123b61e163; root_uuid c2956866-50a0-4e52-8385-61296f5ada12 -> 27c31603-b2e8-4b1a-86a9-80123b61e163
Changed lines of the file:
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@@
 			)
 		)
-		(property "hierarchy_path" "/c2956866-50a0-4e52-8385-61296f5ada12"
+		(property "hierarchy_path" "/27c31603-b2e8-4b1a-86a9-80123b61e163"
 			(at 33.02 40.6399 0)
 			(effects
@@
 			)
 		)
-		(property "root_uuid" "c2956866-50a0-4e52-8385-61296f5ada12"
+		(property "root_uuid" "27c31603-b2e8-4b1a-86a9-80123b61e163"
 			(at 33.02 40.6399 0)
 			(effects
@@
 		(instances
 			(project "two_resistors_connected"
-				(path "/c2956866-50a0-4e52-8385-61296f5ada12"
+				(path "/27c31603-b2e8-4b1a-86a9-80123b61e163"
 					(reference "R1")
 					(unit 1)
@@
 			)
 		)
-		(property "hierarchy_path" "/c2956866-50a0-4e52-8385-61296f5ada12"
+		(property "hierarchy_path" "/27c31603-b2e8-4b1a-86a9-80123b61e163"
 			(at 58.42 40.6399 0)
 			(effects
@@
 			)
 		)
-		(property "root_uuid" "c2956866-50a0-4e52-8385-61296f5ada12"
+		(property "root_uuid" "27c31603-b2e8-4b1a-86a9-80123b61e163"
 			(at 58.42 40.6399 0)
 			(effects
@@
 		(instances
 			(project "two_resistors_connected"
-				(path "/c2956866-50a0-4e52-8385-61296f5ada12"
+				(path "/27c31603-b2e8-4b1a-86a9-80123b61e163"
 					(reference "R2")
 					(unit 1)
