File: tests/bidirectional/37_replace_subcircuit_contents/subcircuit_redesign/subcircuit_redesign.kicad_sch (KiCad schematic)
At the start: 1 part

Commit message: fix: Complete test 37 hierarchical subcircuit redesign
Test 37: Replace subcircuit contents - WORKING

## Changes

### Fixture (subcircuit_redesign.py)
- Two @circuit decorated functions: amplifier_subcircuit() and subcircuit_redesign()
- Root circuit calls amplifier_subcircuit() to create hierarchy
- Clean comment/uncomment pattern for manual testing
- Initial: R1 (10k), C1 (1µF) in subcircuit
- Modified: R2 (22k), R3 (47k), C2 (10µF) in subcircuit

### Test Files
- Updated test to expect amplifier_subcircuit_1.kicad_sch
- Fixed comment/uncomment replacements for all components
- Updated JSON validation for amplifier_subcircuit_1

### Documentation (BIDIRECTIONAL_TEST_SUMMARY.md)
- Updated progress: 28 → 29 tests (41% → 43%)
- Documented test 37 as PASSING
- Notes: Synchronization falls back to regeneration (acceptable)

## Manual Testing Confirmed

**Initial generation:**
- Root: R_main1 (1 component)
- Child: amplifier_subcircuit_1 with R1, C1

**After redesign:**
- Root: R_main1 (unchanged)
- Child: amplifier_subcircuit_1 with R2, R3, C2
- Old components removed, new components added

## What This Validates

**Critical hierarchical workflow:**
- Create circuit with subcircuit module
- Redesign internals of subcircuit module
- Root circuit unaffected by subcircuit changes
- Hierarchical structure preserved
- Different from tests 34/35 (flat bulk operations)

🤖 Generated with [Claude Code](https://claude.com/claude-code)

Co-Authored-By: Claude <noreply@anthropic.com>
Parts:
- R_main1: hierarchy_path /e3d1383c-0168-49f1-9828-030748e2ecf2 -> /ec8ca999-376f-408a-b1e2-c06b980c8b82; root_uuid e3d1383c-0168-49f1-9828-030748e2ecf2 -> ec8ca999-376f-408a-b1e2-c06b980c8b82
Changed lines of the file:
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@@
 			)
 		)
-		(property "hierarchy_path" "/e3d1383c-0168-49f1-9828-030748e2ecf2"
+		(property "hierarchy_path" "/ec8ca999-376f-408a-b1e2-c06b980c8b82"
 			(at 99.06 40.6399 0)
 			(effects
@@
 			)
 		)
-		(property "root_uuid" "e3d1383c-0168-49f1-9828-030748e2ecf2"
+		(property "root_uuid" "ec8ca999-376f-408a-b1e2-c06b980c8b82"
 			(at 99.06 40.6399 0)
 			(effects
@@
 		(instances
 			(project "subcircuit_redesign"
-				(path "/e3d1383c-0168-49f1-9828-030748e2ecf2"
+				(path "/ec8ca999-376f-408a-b1e2-c06b980c8b82"
 					(reference "R_main1")
 					(unit 1)
@@
 		(instances
 			(project "subcircuit_redesign"
-				(path "/e3d1383c-0168-49f1-9828-030748e2ecf2"
+				(path "/ec8ca999-376f-408a-b1e2-c06b980c8b82"
 					(page "2")
 				)
